File: SolarAdapter.kicad_sch (KiCad schematic)
At the start: 7 parts, among them J1 Conn_02x03_Odd_Even, J2 USB_A

Commit message: Solar Adapter 1.1
Release Notes:
1. Added MPNs to parts(whoops)
2. Beefed up power traces to allow for higher current draws
Parts:
- J1: MPN (none) -> FTSH-103-04-L-DH
- J2: MPN (none) -> 6364372-2
- JP1, JP2, JP3, JP4: now left out of the parts list
- R1: MPN (none) -> ERJ-PA3F1004V
Changed lines of the file:
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@@
+			)
+		)
+		(property "MPN" "ERJ-PA3F1004V"
+			(at 124.46 107.95 0)
+			(effects
+				(font
+					(size 1.27 1.27)
+				)
+				(hide yes)
 			)
 		)
@@
 		(unit 1)
 		(exclude_from_sim no)
-		(in_bom yes)
+		(in_bom no)
 		(on_board yes)
 		(dnp no)
@@
 			)
 		)
+		(property "MPN" "FTSH-103-04-L-DH"
+			(at 161.29 96.52 0)
+			(effects
+				(font
+					(size 1.27 1.27)
+				)
+				(hide yes)
+			)
+		)
 		(pin "6"
 		)
@@
 			)
 		)
+		(property "MPN" "6364372-2"
+			(at 127 95.25 0)
+			(effects
+				(font
+					(size 1.27 1.27)
+				)
+				(hide yes)
+			)
+		)
 		(pin "2"
 		)
@@
 		(unit 1)
 		(exclude_from_sim no)
-		(in_bom yes)
+		(in_bom no)
 		(on_board yes)
 		(dnp no)
@@
 		(unit 1)
 		(exclude_from_sim no)
-		(in_bom yes)
+		(in_bom no)
 		(on_board yes)
 		(dnp no)
@@
 		(unit 1)
 		(exclude_from_sim no)
-		(in_bom yes)
-		(on_board yes)
-		(dnp no)
+		(in_bom no)
+		(on_board yes)
+		(dnp no)

Commit message: Solar Adapter 1.1.1
Patch Notes:
1. Original connector was too short, so it was replaced with a longer connector
Parts:
- J1: footprint SolarAdapter:SAMTEC_FTSH-103-04-L-DH -> SolarAdapter:SAMTEC_TMS-103-01-L-D-RA
Changed lines of the file:
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@@
 			)
 		)
-		(property "Footprint" "SolarAdapter:SAMTEC_FTSH-103-04-L-DH"
+		(property "Footprint" "SolarAdapter:SAMTEC_TMS-103-01-L-D-RA"
 			(at 161.29 96.52 0)
 			(effects
